File: io.kicad_sch (KiCad schematic)
At the start: 30 parts

Commit message: schematic: add mezanine interfaces
Connections:
- net PPM_INPUT renamed PPM_IN
Changed lines of the file:
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@@
     (effects (font (size 1.27 1.27)) (justify left))
   )
-  (hierarchical_label "PPM_INPUT" (shape input) (at 105.41 99.06 0)
+  (hierarchical_label "PPM_IN" (shape input) (at 105.41 99.06 0)
     (effects (font (size 1.27 1.27)) (justify left))
   )

Commit message: schematic: update power and fix errors
* specify separate 3V3 lines
* remove bus symbols due to incorrect usage
* pass ERC
Parts:
- gave numbers to parts that had none: 30
Connections:
- net +1V1 renamed 1V1
- net +3V3 renamed 3V3_IO
Other:
- note added: "RP2040 IO MCU"
- note removed: "RP2040 Main MCU"
- moved on the sheet: C40

Commit message: add footprint assignments
Parts:
- C40: footprint (none) -> Capacitor_SMD:C_0402_1005Metric
- R24, R25: footprint (none) -> Resistor_SMD:R_0402_1005Metric
Changed lines of the file:
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@@
       (effects (font (size 1.27 1.27)) (justify right))
     )
-    (property "Footprint" "" (id 2) (at 166.6748 74.93 0)
+    (property "Footprint" "Capacitor_SMD:C_0402_1005Metric" (id 2) (at 166.6748 74.93 0)
       (effects (font (size 1.27 1.27)) hide)
     )
@@
       (effects (font (size 1.27 1.27)) (justify left))
     )
-    (property "Footprint" "" (id 2) (at 125.222 66.04 90)
+    (property "Footprint" "Resistor_SMD:R_0402_1005Metric" (id 2) (at 125.222 66.04 90)
       (effects (font (size 1.27 1.27)) hide)
     )
@@
       (effects (font (size 1.27 1.27)) (justify left))
     )
-    (property "Footprint" "" (id 2) (at 125.222 85.09 90)
-      (effects (font (size 1.27 1.27)) hide)
-    )
+    (property "Footprint" "Resistor_SMD:R_0402_1005Metric" (id 2) (at 125.222 85.09 90)
+      (effects (font (size 1.27 1.27)) hide)
+    )

Commit message: pcb layout draft, incomplete
Parts:
- removed C30: 0.1uF, Capacitor_SMD:C_0402_1005Metric, symbol Device:C
- removed TP4: QSPI_SS, TestPoint:TestPoint_Pad_D1.0mm, symbol Connector:TestPoint
- removed Y2: 12MHz, Crystal:Crystal_SMD_3225-4Pin_3.2x2.5mm, symbol Device:Crystal
- added C44: 0.1uF, Capacitor_SMD:C_0402_1005Metric, symbol Device:C
- added Y2: 12MHz, Crystal:Crystal_SMD_2520-4Pin_2.5x2.0mm, symbol Device:Crystal_GND24
- R22: value 10K -> 1K
- TP5: value TestPoint -> IO_QSPI_SCK
- TP6: value TestPoint -> IO_QSPI_SD3
- U7: value W25Q32JWUU -> W25Q16JVUX; footprint USON:USON8 -> USON:8-USON
Connections:
- net 3V3_IO: now also C44.1
- net GND: now also C44.2, Y2.2, Y2.4
- net LED_AMBER: now also U6.30 (GPIO19); no longer U6.18 (GPIO15)
- net LED_GREEN: now also U6.29 (GPIO18); no longer U6.17 (GPIO14)
- net UART0_RX_FMU: now also U6.41 (GPIO29_ADC3); no longer U6.16 (GPIO13)
- net UART0_TX_FMU: now also U6.40 (GPIO28_ADC2); no longer U6.15 (GPIO12)
- net XIN: now also Y2.1
- net XOUT: now also Y2.3
- net BOOTSEL: now reaches R22.1
- net BOOTSEL: no longer R21.2
- net QSPI_SCLK renamed QSPI_SCK
- net QSPI_SS renamed QSPI_nCS
- net QSPI_nCS: now also R21.2
Other:
- moved on the sheet: C39, C41, C42, R21, R22
