File: fmu.kicad_sch (KiCad schematic)
At the start: 44 parts

Commit message: schematic: add mezanine interfaces
Connections:
- net UART1_CTS_GNSS renamed BUZZER
- net UART1_RTS_GNSS renamed GPIO23_RSV
Changed lines of the file:
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@@
-    (effects (font (size 1.27 1.27)) (justify left))
-  )
-  (hierarchical_label "UART1_CTS_GNSS" (shape input) (at 104.14 113.03 0)
     (effects (font (size 1.27 1.27)) (justify left))
   )
   (hierarchical_label "VBAT_SENSE" (shape input) (at 251.46 71.12 0)
+    (effects (font (size 1.27 1.27)) (justify left))
+  )
+  (hierarchical_label "BUZZER" (shape input) (at 104.14 113.03 0)
     (effects (font (size 1.27 1.27)) (justify left))
   )
@@
   )
   (hierarchical_label "UART0_TX_TELEM" (shape input) (at 104.14 97.79 0)
-    (effects (font (size 1.27 1.27)) (justify left))
-  )
-  (hierarchical_label "UART1_RTS_GNSS" (shape input) (at 104.14 115.57 0)
     (effects (font (size 1.27 1.27)) (justify left))
   )
@@
     (effects (font (size 1.27 1.27)) (justify left))
   )
+  (hierarchical_label "GPIO23_RSV" (shape input) (at 104.14 115.57 0)
+    (effects (font (size 1.27 1.27)) (justify left))
+  )

Commit message: schematic: update power and fix errors
* specify separate 3V3 lines
* remove bus symbols due to incorrect usage
* pass ERC
Parts:
- gave numbers to parts that had none: 44
Connections:
- net +1V1 renamed 1V1
- net +3V3 renamed 3V3_FMU
- net 3V3_FMU: no longer J5.4 (VDD)
- new net 3V3_SD: J5.4 (VDD)

Commit message: add footprint assignments
Parts:
- C16, C17, C18, C19: footprint (none) -> Capacitor_SMD:C_0402_1005Metric
- J5: footprint (none) -> Connector_Card:microSD_HC_Hirose_DM3AT-SF-PEJM5
- R14, R15, R16, R17, R18, R4, R5, R6, R7: footprint (none) -> Resistor_SMD:R_0402_1005Metric
- U2: value W25Q32JWUU -> W25Q16JVUX; footprint USON:USON8 -> USON:8-USON
Changed lines of the file:
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@@
     (property "Reference" "R7" (id 0) (at 154.94 132.08 90))
     (property "Value" "47K" (id 1) (at 154.94 134.62 90))
-    (property "Footprint" "" (id 2) (at 154.94 136.398 90)
+    (property "Footprint" "Resistor_SMD:R_0402_1005Metric" (id 2) (at 154.94 136.398 90)
       (effects (font (size 1.27 1.27)) hide)
     )
@@
     (property "Reference" "R17" (id 0) (at 231.14 139.7 90))
     (property "Value" "0R" (id 1) (at 231.14 142.24 90))
-    (property "Footprint" "" (id 2) (at 231.14 144.018 90)
+    (property "Footprint" "Resistor_SMD:R_0402_1005Metric" (id 2) (at 231.14 144.018 90)
       (effects (font (size 1.27 1.27)) hide)
     )
@@
     (property "Reference" "R4" (id 0) (at 154.94 119.38 90))
     (property "Value" "47K" (id 1) (at 154.94 121.92 90))
-    (property "Footprint" "" (id 2) (at 154.94 123.698 90)
+    (property "Footprint" "Resistor_SMD:R_0402_1005Metric" (id 2) (at 154.94 123.698 90)
       (effects (font (size 1.27 1.27)) hide)
     )
@@
     (property "Reference" "R15" (id 0) (at 224.79 76.2 90))
     (property "Value" "1K" (id 1) (at 224.79 73.66 90))
-    (property "Footprint" "" (id 2) (at 224.79 75.438 90)
+    (property "Footprint" "Resistor_SMD:R_0402_1005Metric" (id 2) (at 224.79 75.438 90)
       (effects (font (size 1.27 1.27)) hide)
     )
@@
     (in_bom yes) (on_board yes)
     (property "Reference" "U2" (id 0) (at 93.98 184.15 0))
-    (property "Value" "W25Q32JWUU" (id 1) (at 99.06 166.37 0))
-    (property "Footprint" "USON:USON8" (id 2) (at 91.44 175.26 0)
+    (property "Value" "W25Q16JVUX" (id 1) (at 99.06 166.37 0))
+    (property "Footprint" "USON:8-USON" (id 2) (at 91.44 175.26 0)
       (effects (font (size 1.27 1.27)) hide)
     )
@@
       (effects (font (size 1.27 1.27)) (justify left))
     )
-    (property "Footprint" "" (id 2) (at 249.8852 83.82 0)
+    (property "Footprint" "Capacitor_SMD:C_0402_1005Metric" (id 2) (at 249.8852 83.82 0)
       (effects (font (size 1.27 1.27)) hide)
     )
@@
       (effects (font (size 1.27 1.27)) (justify left))
     )
-    (property "Footprint" "" (id 2) (at 234.442 80.01 90)
+    (property "Footprint" "Resistor_SMD:R_0402_1005Metric" (id 2) (at 234.442 80.01 90)
       (effects (font (size 1.27 1.27)) hide)
     )
@@
     (property "Reference" "R6" (id 0) (at 154.94 127 90))
     (property "Value" "47K" (id 1) (at 154.94 129.54 90))
-    (property "Footprint" "" (id 2) (at 154.94 131.318 90)
+    (property "Footprint" "Resistor_SMD:R_0402_1005Metric" (id 2) (at 154.94 131.318 90)
       (effects (font (size 1.27 1.27)) hide)
     )
@@
       (effects (font (size 1.27 1.27)) (justify left))
     )
-    (property "Footprint" "" (id 2) (at 229.362 80.01 90)
+    (property "Footprint" "Resistor_SMD:R_0402_1005Metric" (id 2) (at 229.362 80.01 90)
       (effects (font (size 1.27 1.27)) hide)
     )
@@
       (effects (font (size 1.27 1.27)) (justify left))
     )
-    (property "Footprint" "" (id 2) (at 230.8352 128.27 0)
+    (property "Footprint" "Capacitor_SMD:C_0402_1005Metric" (id 2) (at 230.8352 128.27 0)
       (effects (font (size 1.27 1.27)) hide)
     )
@@
     (property "Reference" "J5" (id 0) (at 205.105 107.95 0))
     (property "Value" "Micro_SD_Card" (id 1) (at 205.105 110.49 0))
-    (property "Footprint" "" (id 2) (at 233.68 119.38 0)
+    (property "Footprint" "Connector_Card:microSD_HC_Hirose_DM3AT-SF-PEJM5" (id 2) (at 233.68 119.38 0)
       (effects (font (size 1.27 1.27)) hide)
     )
@@
       (effects (font (size 1.27 1.27)) (justify left))
     )
-    (property "Footprint" "" (id 2) (at 238.4552 128.27 0)
+    (property "Footprint" "Capacitor_SMD:C_0402_1005Metric" (id 2) (at 238.4552 128.27 0)
       (effects (font (size 1.27 1.27)) hide)
     )
@@
       (effects (font (size 1.27 1.27)) (justify left))
     )
-    (property "Footprint" "" (id 2) (at 243.5352 83.82 0)
+    (property "Footprint" "Capacitor_SMD:C_0402_1005Metric" (id 2) (at 243.5352 83.82 0)
       (effects (font (size 1.27 1.27)) hide)
     )
@@
     (property "Reference" "R14" (id 0) (at 224.79 68.58 90))
     (property "Value" "1K" (id 1) (at 224.79 71.12 90))
-    (property "Footprint" "" (id 2) (at 224.79 72.898 90)
+    (property "Footprint" "Resistor_SMD:R_0402_1005Metric" (id 2) (at 224.79 72.898 90)
       (effects (font (size 1.27 1.27)) hide)
     )
@@
     (property "Reference" "R5" (id 0) (at 158.75 125.73 90))
     (property "Value" "47K" (id 1) (at 154.94 124.46 90))
-    (property "Footprint" "" (id 2) (at 154.94 126.238 90)
-      (effects (font (size 1.27 1.27)) hide)
-    )
+    (property "Footprint" "Resistor_SMD:R_0402_1005Metric" (id 2) (at 154.94 126.238 90)
+      (effects (font (size 1.27 1.27)) hide)
+    )

Commit message: pcb layout draft, incomplete
Parts:
- removed C4: 0.1uF, Capacitor_SMD:C_0402_1005Metric, symbol Device:C
- removed J5: Micro_SD_Card, Connector_Card:microSD_HC_Hirose_DM3AT-SF-PEJM5, symbol Connector:Micro_SD_Card
- removed TP1: QSPI_SS, TestPoint:TestPoint_Pad_D1.0mm, symbol Connector:TestPoint
- removed Y1: 12MHz, Crystal:Crystal_SMD_3225-4Pin_3.2x2.5mm, symbol Device:Crystal
- added C43: 0.1uF, Capacitor_SMD:C_0402_1005Metric, symbol Device:C
- added J5: Micro_SD_Card_Det_Hirose_DM3AT, Connector_Card:microSD_HC_Hirose_DM3AT-SF-PEJM5, symbol Connector:Micro_SD_Card_Det_Hirose_DM3AT
- added R28, R29: 0R, Resistor_SMD:R_0402_1005Metric, symbol Device:R
- added Y1: 12MHz, Crystal:Crystal_SMD_2520-4Pin_2.5x2.0mm, symbol Device:Crystal_GND24
- R1: value 10K -> 1K
- TP2: value TestPoint -> FMU_QSPI_SCK
- TP3: value TestPoint -> FMU_QSPI_SD3
Connections:
- net QSPI_SS is gone; now on net QSPI_nCS: R2.2, R3.2, U1.56 (QSPI_SS), U2.1 (~{CS})
- net 3V3_FMU: now also R2.1, C43.1; no longer R1.1
- net 3V3_SD: now also J5.4 (VDD)
- net GND: now also C43.2, J5.6 (VSS), J5.9 (DET_B), Y1.2, Y1.4
- net SDMMC_CD: now also R28.1, R29.1
- net SPI1_PICO_SDMMC: now also J5.3 (CMD)
- net SPI1_POCI_SDMMC: now also J5.7 (DAT0)
- net SPI1_SCK_SDMMC: now also J5.5 (CLK)
- net XIN: now also Y1.1
- net XOUT: now also Y1.3
- net at R17.1: now also J5.11 (SHIELD)
- net QSPI_nCS: now reaches R1.2
- net QSPI_nCS: no longer R2.1
- net QSPI_SCLK renamed QSPI_SCK
- new net: J5.10 (DET_A), R29.2
- new net: J5.2 (DAT3/CD), R28.2
- new net BOOTSEL: R1.1
Other:
- moved on the sheet: C13, C7, R17, R3, R4, R5, R6, R7, TP2, TP3, U2

Commit message: layout improvements, connector change
Connections:
- net IBAT_SENSE: now also U1.40 (GPIO28_ADC2); no longer U1.41 (GPIO29_ADC3)
- net VBAT_SENSE: now also U1.41 (GPIO29_ADC3); no longer U1.40 (GPIO28_ADC2)
Changed lines of the file:
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@@
     (effects (font (size 1.27 1.27)) (justify right bottom))
   )
-  (label "IBAT_SENSE" (at 123.19 133.35 180)
+  (label "IBAT_SENSE" (at 123.19 130.81 180)
     (effects (font (size 1.27 1.27)) (justify right bottom))
   )
@@
     (effects (font (size 1.27 1.27)) (justify left bottom))
   )
-  (label "VBAT_SENSE" (at 123.19 130.81 180)
+  (label "VBAT_SENSE" (at 123.19 133.35 180)
     (effects (font (size 1.27 1.27)) (justify right bottom))
   )
