File: microfc-fmu-v3.1.kicad_pcb (KiCad board)
At the start: 2 copper layers, 32 x 26 mm, 88 parts, among them J2 FMU Bus [Top], J4 [IO Bus Top], J5 Micro_SD_Card_Det_Hirose_DM3AT, U1 RP2040, U2 W25Q16JVUX, U3 ICM42605, U4 BMM150, U5 ICP20100, U6 RP2040, U7 W25Q16JVUX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

Commit message: layout improvements, connector change
Parts:
- J2: footprint Hirose_DF40:HIROSE_DF40C-40DS-0.4V(51) -> Hirose_DF12N:HRS_DF12NB(3.0)-40DP-0.5V(51)
- moved C8 13.7 mm to (124.1, 125.1)
- moved R12 11.0 mm to (124.5, 120.2)
- moved R13 11.0 mm to (124.5, 121.3)
- moved R1 8.72 mm to (133.7, 91.8)
- moved R3 8.72 mm to (127.0, 91.8)
- moved TP2 8.72 mm to (124.4, 90.1)
- moved C43 8.72 mm to (132.9, 96.8)
- moved C7 8.72 mm to (129.2, 91.8)
- moved R10 8.72 mm to (134.8, 101.9)
- moved R11 8.72 mm to (134.8, 103.0)
- moved R2 8.72 mm to (133.1, 90.2)
- moved TP3 8.72 mm to (129.6, 89.5)
- moved C44 5.70 mm to (105.7, 114.6)
- moved R22 2.04 mm to (102.8, 106.3), turned to 90 degrees
- moved J2 1.36 mm to (130.3, 113.2), turned to -90 degrees
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Routing:
- net /SAFETY_LED: track 0.00 -> 2.75 mm
- net /SAFETY_SWITCH: track 0.00 -> 2.75 mm
- net /IO_CH4: track 0.00 -> 2.75 mm
- net /IO_CH3: track 0.00 -> 2.75 mm
- net /IO_CH2: track 0.00 -> 2.75 mm
- net /IO_CH1: track 0.00 -> 2.75 mm
- net /IO_CH5: track 0.00 -> 2.59 mm
- net /IO_CH7: track 0.00 -> 2.59 mm
- net /IO_CH8: track 0.00 -> 2.59 mm
- net /IO_CH6: track 0.00 -> 2.59 mm
- net /3V3_FMU: track 12.1 -> 9.50 mm
- net /IO Processor/1V1: track 6.77 -> 5.07 mm
- net /FMU_CH4: track 0.00 -> 1.62 mm, vias 0 -> 1
- net /IO_LED_BLUE: track 0.00 -> 1.52 mm, vias 0 -> 2
- net /IO_SWDIO: track 0.00 -> 1.42 mm, vias 0 -> 2
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