File: microfc-fmu-v3.1.kicad_sch (KiCad schematic)
At the start: 4 parts, among them J1 FMU Bus [Bottom], J2 FMU Bus [Top], J3 [IO Bus Bottom], J4 [IO Bus Top]

Commit message: add footprint assignments
Parts:
- J1, J3: footprint (none) -> Hirose_DF40:HRS_DF40C-40DP-0.4V(51)
- J2, J4: footprint (none) -> Hirose_DF40:DF40C-40DS-0.4V
Changed lines of the file:
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@@
     (property "Reference" "J3" (id 0) (at 166.37 93.98 0))
     (property "Value" "[IO Bus Bottom]" (id 1) (at 166.37 96.52 0))
-    (property "Footprint" "" (id 2) (at 165.1 123.19 0)
+    (property "Footprint" "Hirose_DF40:HRS_DF40C-40DP-0.4V(51)" (id 2) (at 165.1 123.19 0)
       (effects (font (size 1.27 1.27)) hide)
     )
@@
     (property "Reference" "J1" (id 0) (at 53.34 93.98 0))
     (property "Value" "FMU Bus [Bottom]" (id 1) (at 53.34 96.52 0))
-    (property "Footprint" "" (id 2) (at 52.07 123.19 0)
+    (property "Footprint" "Hirose_DF40:HRS_DF40C-40DP-0.4V(51)" (id 2) (at 52.07 123.19 0)
       (effects (font (size 1.27 1.27)) hide)
     )
@@
     (property "Reference" "J4" (id 0) (at 218.44 93.98 0))
     (property "Value" "[IO Bus Top]" (id 1) (at 218.44 96.52 0))
-    (property "Footprint" "" (id 2) (at 217.17 123.19 0)
+    (property "Footprint" "Hirose_DF40:DF40C-40DS-0.4V" (id 2) (at 217.17 123.19 0)
       (effects (font (size 1.27 1.27)) hide)
     )
@@
     (property "Reference" "J2" (id 0) (at 105.41 93.98 0))
     (property "Value" "FMU Bus [Top]" (id 1) (at 105.41 96.52 0))
-    (property "Footprint" "" (id 2) (at 104.14 123.19 0)
+    (property "Footprint" "Hirose_DF40:DF40C-40DS-0.4V" (id 2) (at 104.14 123.19 0)
       (effects (font (size 1.27 1.27)) hide)
     )
@@
     )
     (path "/b7f4c42a-ec09-47f5-88b3-96098e35479a/a5621010-98c1-4d72-9273-5a31fa595113"
-      (reference "C16") (unit 1) (value "2.2uF") (footprint "")
+      (reference "C16") (unit 1) (value "2.2uF") (footprint "Capacitor_SMD:C_0402_1005Metric")
     )
     (path "/b7f4c42a-ec09-47f5-88b3-96098e35479a/c42da642-38aa-4fad-921c-a0441865802e"
-      (reference "C17") (unit 1) (value "0.1uF") (footprint "")
+      (reference "C17") (unit 1) (value "0.1uF") (footprint "Capacitor_SMD:C_0402_1005Metric")
     )
     (path "/b7f4c42a-ec09-47f5-88b3-96098e35479a/c6d4a150-742b-4b94-b89c-9540e247c717"
-      (reference "C18") (unit 1) (value "0.1uF") (footprint "")
+      (reference "C18") (unit 1) (value "0.1uF") (footprint "Capacitor_SMD:C_0402_1005Metric")
     )
     (path "/b7f4c42a-ec09-47f5-88b3-96098e35479a/722a724d-3db5-45f5-9ee8-c6f9485bd809"
-      (reference "C19") (unit 1) (value "0.1uF") (footprint "")
+      (reference "C19") (unit 1) (value "0.1uF") (footprint "Capacitor_SMD:C_0402_1005Metric")
     )
     (path "/b7f4c42a-ec09-47f5-88b3-96098e35479a/52dd5bf7-d865-475e-99f4-3dd6a1b4d2f7/b18783e8-7516-4abb-9af3-c9a77a24d23e"
@@
     )
     (path "/b7f4c42a-ec09-47f5-88b3-96098e35479a/52dd5bf7-d865-475e-99f4-3dd6a1b4d2f7/a432fbc5-fe1d-4e84-af9c-4098473d40d4"
-      (reference "C23") (unit 1) (value "0.1uF") (footprint "")
+      (reference "C23") (unit 1) (value "0.1uF") (footprint "Capacitor_SMD:C_0402_1005Metric")
     )
     (path "/b7f4c42a-ec09-47f5-88b3-96098e35479a/52dd5bf7-d865-475e-99f4-3dd6a1b4d2f7/6c51f962-df95-4e4a-a3e3-379acfecc1e1"
-      (reference "C24") (unit 1) (value "0.1uF") (footprint "")
+      (reference "C24") (unit 1) (value "0.1uF") (footprint "Capacitor_SMD:C_0402_1005Metric")
     )
     (path "/b7f4c42a-ec09-47f5-88b3-96098e35479a/52dd5bf7-d865-475e-99f4-3dd6a1b4d2f7/a7ed50f3-df4c-4ed9-b295-8360deaeb8dd"
@@
     )
     (path "/3afd19d3-a8af-488e-befe-c9bfd85f2b97/07675f38-af39-4a2d-b938-68204d7e8bc4"
-      (reference "C40") (unit 1) (value "0.1uF") (footprint "")
+      (reference "C40") (unit 1) (value "0.1uF") (footprint "Capacitor_SMD:C_0402_1005Metric")
     )
     (path "/3afd19d3-a8af-488e-befe-c9bfd85f2b97/0d51e0e3-f387-4fa3-bc98-5ddb68db701e"
@@
     )
     (path "/9c0865a7-183b-46e2-a256-b53ccfae1a8e"
-      (reference "J1") (unit 1) (value "FMU Bus [Bottom]") (footprint "")
+      (reference "J1") (unit 1) (value "FMU Bus [Bottom]") (footprint "Hirose_DF40:HRS_DF40C-40DP-0.4V(51)")
     )
     (path "/f9937900-c7e9-484c-8c19-08a1486cee80"
-      (reference "J2") (unit 1) (value "FMU Bus [Top]") (footprint "")
+      (reference "J2") (unit 1) (value "FMU Bus [Top]") (footprint "Hirose_DF40:DF40C-40DS-0.4V")
     )
     (path "/5ae7b426-6c30-416b-966f-159e60bf5e37"
-      (reference "J3") (unit 1) (value "[IO Bus Bottom]") (footprint "")
+      (reference "J3") (unit 1) (value "[IO Bus Bottom]") (footprint "Hirose_DF40:HRS_DF40C-40DP-0.4V(51)")
     )
     (path "/a1782542-3abe-4344-b418-7870c468beab"
-      (reference "J4") (unit 1) (value "[IO Bus Top]") (footprint "")
+      (reference "J4") (unit 1) (value "[IO Bus Top]") (footprint "Hirose_DF40:DF40C-40DS-0.4V")
     )
     (path "/b7f4c42a-ec09-47f5-88b3-96098e35479a/aca8d602-9482-4cef-8c60-7c037cad9604"
-      (reference "J5") (unit 1) (value "Micro_SD_Card") (footprint "")
+      (reference "J5") (unit 1) (value "Micro_SD_Card") (footprint "Connector_Card:microSD_HC_Hirose_DM3AT-SF-PEJM5")
     )
     (path "/b7f4c42a-ec09-47f5-88b3-96098e35479a/7d6a3251-6a50-4ab1-b0ef-b9418f48d1fb"
@@
     )
     (path "/b7f4c42a-ec09-47f5-88b3-96098e35479a/4cb13a80-0fe3-4a7a-b433-5c0aa8658149"
-      (reference "R4") (unit 1) (value "47K") (footprint "")
+      (reference "R4") (unit 1) (value "47K") (footprint "Resistor_SMD:R_0402_1005Metric")
     )
     (path "/b7f4c42a-ec09-47f5-88b3-96098e35479a/cff12ead-0c13-4eb6-b473-c0d5e0a06d31"
-      (reference "R5") (unit 1) (value "47K") (footprint "")
+      (reference "R5") (unit 1) (value "47K") (footprint "Resistor_SMD:R_0402_1005Metric")
     )
     (path "/b7f4c42a-ec09-47f5-88b3-96098e35479a/8a0b4fb7-a70b-4796-b11c-270544ed1da7"
-      (reference "R6") (unit 1) (value "47K") (footprint "")
+      (reference "R6") (unit 1) (value "47K") (footprint "Resistor_SMD:R_0402_1005Metric")
     )
     (path "/b7f4c42a-ec09-47f5-88b3-96098e35479a/010b1ed3-32fe-4364-8f6e-f34ec963bccb"
-      (reference "R7") (unit 1) (value "47K") (footprint "")
+      (reference "R7") (unit 1) (value "47K") (footprint "Resistor_SMD:R_0402_1005Metric")
     )
     (path "/b7f4c42a-ec09-47f5-88b3-96098e35479a/381d592c-3e87-4ec8-881f-c7c3f16268f4"
@@
     )
     (path "/b7f4c42a-ec09-47f5-88b3-96098e35479a/c7862db2-be2a-478f-8a12-8bf7200e8607"
-      (reference "R14") (unit 1) (value "1K") (footprint "")
+      (reference "R14") (unit 1) (value "1K") (footprint "Resistor_SMD:R_0402_1005Metric")
     )
     (path "/b7f4c42a-ec09-47f5-88b3-96098e35479a/5859ff60-3859-459f-9840-add68a808e71"
-      (reference "R15") (unit 1) (value "1K") (footprint "")
+      (reference "R15") (unit 1) (value "1K") (footprint "Resistor_SMD:R_0402_1005Metric")
     )
     (path "/b7f4c42a-ec09-47f5-88b3-96098e35479a/a1ef9828-8708-489b-9306-f8a0394aa8a6"
-      (reference "R16") (unit 1) (value "1M") (footprint "")
+      (reference "R16") (unit 1) (value "1M") (footprint "Resistor_SMD:R_0402_1005Metric")
     )
     (path "/b7f4c42a-ec09-47f5-88b3-96098e35479a/0ad0806f-84aa-4b26-8df2-2d541503024d"
-      (reference "R17") (unit 1) (value "0R") (footprint "")
+      (reference "R17") (unit 1) (value "0R") (footprint "Resistor_SMD:R_0402_1005Metric")
     )
     (path "/b7f4c42a-ec09-47f5-88b3-96098e35479a/7a735e77-2b56-40d1-8cd0-20a198ef72ce"
-      (reference "R18") (unit 1) (value "1M") (footprint "")
+      (reference "R18") (unit 1) (value "1M") (footprint "Resistor_SMD:R_0402_1005Metric")
     )
     (path "/b7f4c42a-ec09-47f5-88b3-96098e35479a/52dd5bf7-d865-475e-99f4-3dd6a1b4d2f7/0d4593f4-135f-4593-a864-0e3e7faf460c"
-      (reference "R19") (unit 1) (value "10K") (footprint "")
+      (reference "R19") (unit 1) (value "10K") (footprint "Resistor_SMD:R_0402_1005Metric")
     )
     (path "/b7f4c42a-ec09-47f5-88b3-96098e35479a/52dd5bf7-d865-475e-99f4-3dd6a1b4d2f7/df951b9d-cd00-41d7-be73-71042fd1e693"
@@
     )
     (path "/3afd19d3-a8af-488e-befe-c9bfd85f2b97/949e50af-2468-4433-aae6-a0df6d7be6e8"
-      (reference "R24") (unit 1) (value "0R [DNP]") (footprint "")
+      (reference "R24") (unit 1) (value "0R [DNP]") (footprint "Resistor_SMD:R_0402_1005Metric")
     )
     (path "/3afd19d3-a8af-488e-befe-c9bfd85f2b97/a7fdf7b4-ca99-44b3-b49f-149d2c5a31f3"
-      (reference "R25") (unit 1) (value "100K") (footprint "")
+      (reference "R25") (unit 1) (value "100K") (footprint "Resistor_SMD:R_0402_1005Metric")
     )
     (path "/3afd19d3-a8af-488e-befe-c9bfd85f2b97/bcf9a619-ff0b-4cdb-898e-f0f20f6e9a2f"
@@
     )
     (path "/b7f4c42a-ec09-47f5-88b3-96098e35479a/70f8aec7-663f-4b07-bb8d-9e5a2c690f71"
-      (reference "U2") (unit 1) (value "W25Q32JWUU") (footprint "USON:USON8")
+      (reference "U2") (unit 1) (value "W25Q16JVUX") (footprint "USON:8-USON")
     )
     (path "/b7f4c42a-ec09-47f5-88b3-96098e35479a/52dd5bf7-d865-475e-99f4-3dd6a1b4d2f7/6700f17a-8aa2-4fa0-b189-f5a32b1146ff"

Commit message: pcb layout draft, incomplete
Parts:
- J2, J4: footprint Hirose_DF40:DF40C-40DS-0.4V -> Hirose_DF40:HIROSE_DF40C-40DS-0.4V(51)
Connections:
- net FMU_RSV6 is gone; now on net FMU_RSV5: J1.38 (Pin_38), J2.38 (Pin_38)
- net I2C1_SCL_EXT is gone; now on net GND: J1.13 (Pin_13), J1.19 (Pin_19), J1.23 (Pin_23), J1.25 (Pin_25), J1.35 (Pin_35), J2.13 (Pin_13), J2.19 (Pin_19), J2.23 (Pin_23), J2.25 (Pin_25), J2.35 (Pin_35)
- net IO_RSV2 is gone; now on net IO_RSV1: J3.38 (Pin_38), J4.38 (Pin_38)
- net FMU_RSV1: now also J1.30 (Pin_30), J2.30 (Pin_30); no longer J1.28 (Pin_28), J2.28 (Pin_28)
- net FMU_RSV2: now also J1.32 (Pin_32), J2.32 (Pin_32); no longer J1.30 (Pin_30), J2.30 (Pin_30)
- net FMU_RSV3: now also J1.34 (Pin_34), J2.34 (Pin_34); no longer J1.32 (Pin_32), J2.32 (Pin_32)
- net FMU_RSV4: now also J1.36 (Pin_36), J2.36 (Pin_36); no longer J1.34 (Pin_34), J2.34 (Pin_34)
- net FMU_RSV5: no longer J1.36 (Pin_36), J2.36 (Pin_36)
- net FMU_SWCLK: now also J1.26 (Pin_26), J2.26 (Pin_26); no longer J1.24 (Pin_24), J2.24 (Pin_24)
- net FMU_SWDIO: now also J1.24 (Pin_24), J2.24 (Pin_24); no longer J1.22 (Pin_22), J2.22 (Pin_22)
- net GND: now also J1.28 (Pin_28), J2.28 (Pin_28), J3.36 (Pin_36), J4.36 (Pin_36); no longer J1.26 (Pin_26), J2.26 (Pin_26), J3.34 (Pin_34), J4.34 (Pin_34)
- net IO_RSV1: no longer J3.36 (Pin_36), J4.36 (Pin_36)
- net IO_SWCLK: now also J3.34 (Pin_34), J4.34 (Pin_34); no longer J3.32 (Pin_32), J4.32 (Pin_32)
- net IO_SWDIO: now also J3.32 (Pin_32), J4.32 (Pin_32); no longer J3.30 (Pin_30), J4.30 (Pin_30)
- new net FMU_BOOTSEL: J1.22 (Pin_22), J2.22 (Pin_22)
- new net IO_BOOTSEL: J3.30 (Pin_30), J4.30 (Pin_30)
Other:
- sheet FMU Processor ports: added BOOTSEL; removed none
- sheet IO Processor ports: added BOOTSEL; removed none

Commit message: layout improvements, connector change
Changed lines of the file:
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@@
   (junction (at 227.33 130.81) (diameter 0) (color 0 0 0 0)
+  )
+  (junction (at 96.52 148.59) (diameter 0) (color 0 0 0 0)
   )
   (junction (at 44.45 148.59) (diameter 0) (color 0 0 0 0)
@@
   )
   (junction (at 175.26 143.51) (diameter 0) (color 0 0 0 0)
+  )
+  (junction (at 96.52 143.51) (diameter 0) (color 0 0 0 0)
   )
   (junction (at 180.34 107.95) (diameter 0) (color 0 0 0 0)
@@
     (stroke (width 0) (type default) (color 0 0 0 0))
   )
+  (wire (pts (xy 96.52 143.51) (xy 96.52 148.59))
+    (stroke (width 0) (type default) (color 0 0 0 0))
+  )
