File: sensors.kicad_sch (KiCad schematic)
At the start: 12 parts

Commit message: schematic: update power and fix errors
* specify separate 3V3 lines
* remove bus symbols due to incorrect usage
* pass ERC
Parts:
- removed U?: ICP20100, ICP20100:PQFN50P200X200X85-10N, symbol ICP20100:ICP20100
- added U5: ICP20100, ICP20100:PQFN50P200X200X85-10N, symbol Invensense_ICP:ICP20100
- gave numbers to parts that had none: 11
Connections:
- net GND: now also U5.3 (VSS), U5.8 (RESV), U5.9 (RESV)
- net SCL: now also U5.2 (SCL/SCLK)
- net SDA: now also U5.4 (SDA/SDI)
- net VDD: now also U5.1 (CSB), U5.10 (VDDIO), U5.5 (VDD)
- net at R20.2: now also U5.6 (AD0/SDO)
- net at U3.10 (RESV): no longer U3.11 (RESV)
- net at U3.2 (RESV): no longer U3.3 (RESV)

Commit message: add footprint assignments
Parts:
- C23, C24: footprint (none) -> Capacitor_SMD:C_0402_1005Metric
- R19: footprint (none) -> Resistor_SMD:R_0402_1005Metric
Changed lines of the file:
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@@
       (effects (font (size 1.27 1.27)) (justify left))
     )
-    (property "Footprint" "" (id 2) (at 68.072 68.58 90)
+    (property "Footprint" "Resistor_SMD:R_0402_1005Metric" (id 2) (at 68.072 68.58 90)
       (effects (font (size 1.27 1.27)) hide)
     )
@@
     (property "Reference" "C24" (id 0) (at 166.37 35.56 90))
     (property "Value" "0.1uF" (id 1) (at 166.37 38.1 90))
-    (property "Footprint" "" (id 2) (at 170.18 42.2148 0)
+    (property "Footprint" "Capacitor_SMD:C_0402_1005Metric" (id 2) (at 170.18 42.2148 0)
       (effects (font (size 1.27 1.27)) hide)
     )
@@
     (property "Reference" "C23" (id 0) (at 151.13 35.56 90))
     (property "Value" "0.1uF" (id 1) (at 151.13 38.1 90))
-    (property "Footprint" "" (id 2) (at 154.94 42.2148 0)
-      (effects (font (size 1.27 1.27)) hide)
-    )
+    (property "Footprint" "Capacitor_SMD:C_0402_1005Metric" (id 2) (at 154.94 42.2148 0)
+      (effects (font (size 1.27 1.27)) hide)
+    )

Commit message: layout improvements, connector change
Parts:
- C20: value 2.2uF -> (none); footprint Capacitor_SMD:C_0402_1005Metric -> (none)
- C21, C23, C24, C25, C26: value 0.1uF -> (none); footprint Capacitor_SMD:C_0402_1005Metric -> (none)
- C22: value 10nF -> (none); footprint Capacitor_SMD:C_0402_1005Metric -> (none)
- R19, R20: value 10K -> (none); footprint Resistor_SMD:R_0402_1005Metric -> (none)
- U3: value ICM42605 -> (none); footprint Package_LGA:LGA-14_3x2.5mm_P0.5mm_LayoutBorder3x4y -> (none)
- U4: value BMM150 -> (none); footprint Package_CSP:WLCSP-12_1.56x1.56mm_P0.4mm -> (none)
- U5: value ICP20100 -> (none); footprint ICP20100:PQFN50P200X200X85-10N -> (none)
